File: Tiramisu.kicad_pcb (KiCad board)
At the start: 2 copper layers, 24 x 32 mm, 26 parts, among them J1 Conn_ARM_SWD_TagConnect_TC203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, J2 USB_C_Receptacle_USB2.0_16P, Q1 Q_PMOS_GSD, U1 MDBT50Q-1MV2, U2 LSM6DSV, U3 MCP73831-2-OT

Commit message: that should be a +3V3 route oops
Connections:
- J1 pad 1: VCC -> +3.3V
Routing:
- net VCC: track 63.9 -> 7.47 mm, vias 2 -> 0
- net +3.3V: track 38.8 -> 42.2 mm
Changed lines of the file:
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@@
 			(size 0.7874 0.7874)
 			(layers "F.Cu" "F.Mask")
-			(net 66 "VCC")
+			(net 62 "+3.3V")
 			(pinfunction "VCC")
 			(pintype "power_in")
@@
 	)
 	(segment
-		(start 111.883027 60.649432)
-		(end 113.332459 59.2)
+		(start 116.9 58.9)
+		(end 117 58.8)
 		(width 0.25)
 		(layer "F.Cu")
@@
 	)
 	(segment
-		(start 116.6 59.2)
-		(end 117 58.8)
-		(width 0.25)
-		(layer "F.Cu")
-		(net 5)
-	)
-	(segment
 		(start 117 58.8)
 		(end 117 57.67)
@@
 		(net 5)
 	)
-	(segment
-		(start 113.332459 59.2)
-		(end 116.6 59.2)
-		(width 0.25)
-		(layer "F.Cu")
-		(net 5)
-	)
-	(segment
-		(start 111.8 60.649432)
-		(end 111.883027 60.649432)
-		(width 0.25)
-		(layer "F.Cu")
-		(net 5)
-	)
 	(via
 		(at 109.05 61.45)
@@
 	)
 	(via
-		(at 111.8 60.649432)
+		(at 116.9 58.9)
 		(size 0.8)
 		(drill 0.4)
@@
 	)
 	(segment
-		(start 109.850568 60.649432)
-		(end 109.05 61.45)
+		(start 115.150568 60.649432)
+		(end 109.850568 60.649432)
 		(width 0.25)
 		(layer "B.Cu")
@@
 	)
 	(segment
-		(start 111.8 60.649432)
-		(end 109.850568 60.649432)
+		(start 116.9 58.9)
+		(end 115.150568 60.649432)
+		(width 0.25)
+		(layer "B.Cu")
+		(net 5)
+	)
+	(segment
+		(start 109.850568 60.649432)
+		(end 109.05 61.45)
 		(width 0.25)
 		(layer "B.Cu")
@@
 	)
 	(segment
+		(start 115.73 60.045)
+		(end 115 60.775)
+		(width 0.25)
+		(layer "F.Cu")
+		(net 62)
+	)
+	(segment
 		(start 119.4 65.125)
 		(end 119.4 66.061956)
@@
 	)
 	(segment
+		(start 115.73 57.67)
+		(end 115.73 60.045)
+		(width 0.25)
+		(layer "F.Cu")
+		(net 62)
+	)
+	(segment
 		(start 116.2 66.8)
 		(end 115 66.8)
@@
 	)
 	(segment
-		(start 102.2 75.2)
-		(end 102.2 70.8)
-		(width 0.25)
-		(layer "F.Cu")
-		(net 66)
-	)
-	(segment
-		(start 121 57.1807)
-		(end 122.725 58.9057)
-		(width 0.25)
-		(layer "F.Cu")
-		(net 66)
-	)
-	(segment
 		(start 107.4375 70.05)
 		(end 107.6 70.2125)
@@
 	)
 	(segment
-		(start 102.2 70.8)
-		(end 102.95 70.05)
-		(width 0.25)
-		(layer "F.Cu")
-		(net 66)
-	)
-	(segment
 		(start 108.6 67.125)
 		(end 108.6 65.6)
@@
 	)
 	(segment
-		(start 102.95 70.05)
-		(end 105.7375 70.05)
-		(width 0.25)
-		(layer "F.Cu")
-		(net 66)
-	)
-	(segment
 		(start 109.225 67.75)
 		(end 108.6 67.125)
@@
 	)
 	(segment
-		(start 122.725 75.475)
-		(end 121.3 76.9)
-		(width 0.25)
-		(layer "F.Cu")
-		(net 66)
-	)
-	(segment
-		(start 119 78.2)
-		(end 120.3 76.9)
-		(width 0.25)
-		(layer "F.Cu")
-		(net 66)
-	)
-	(segment
-		(start 119 78.2)
-		(end 105.2 78.2)
-		(width 0.25)
-		(layer "F.Cu")
-		(net 66)
-	)
-	(segment
-		(start 122.725 58.9057)
-		(end 122.725 75.475)
-		(width 0.25)
-		(layer "F.Cu")
-		(net 66)
-	)
-	(segment
-		(start 116.375 58.315)
-		(end 115.73 57.67)
-		(width 0.25)
-		(layer "F.Cu")
-		(net 66)
-	)
-	(segment
 		(start 108.178125 69.634375)
 		(end 108.178125 68.796875)
@@
 	)
 	(segment
-		(start 116.375 58.4)
-		(end 116.375 58.315)
-		(width 0.25)
-		(layer "F.Cu")
-		(net 66)
-	)
-	(segment
 		(start 107.6 70.2125)
 		(end 108.178125 69.634375)
@@
 		(net 66)
 	)
-	(segment
-		(start 105.2 78.2)
-		(end 102.2 75.2)
-		(width 0.25)
-		(layer "F.Cu")
-		(net 66)
-	)
-	(segment
-		(start 120.3 76.9)
-		(end 121.3 76.9)
-		(width 0.25)
-		(layer "F.Cu")
-		(net 66)
-	)
-	(via
-		(at 116.375 58.4)
-		(size 0.6)
-		(drill 0.3)
-		(layers "F.Cu" "B.Cu")
-		(net 66)
-	)
-	(via
-		(at 121 57.1807)
-		(size 0.6)
-		(drill 0.3)
-		(layers "F.Cu" "B.Cu")
-		(net 66)
-	)
-	(segment
-		(start 120.8193 57)
-		(end 121 57.1807)
-		(width 0.25)
-		(layer "B.Cu")
-		(net 66)
-	)
-	(segment
-		(start 117.775 57)
-		(end 120.8193 57)
-		(width 0.25)
-		(layer "B.Cu")
-		(net 66)
-	)
-	(segment
-		(start 116.375 58.4)
-		(end 117.775 57)
-		(width 0.25)
-		(layer "B.Cu")
-		(net 66)
-	)

Commit message: final export
Parts:
- H1, H2, H3: footprint adhoc:MountingHole_1.8mm_M1.6 -> adhoc:MountingHole_1.7mm_M1.6
Changed lines of the file:
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@@
 			(plot_on_all_layers_selection 0x0000000_00000000)
 			(disableapertmacros no)
-			(usegerberextensions no)
-			(usegerberattributes yes)
-			(usegerberadvancedattributes yes)
-			(creategerberjobfile yes)
+			(usegerberextensions yes)
+			(usegerberattributes no)
+			(usegerberadvancedattributes no)
+			(creategerberjobfile no)
 			(dashed_line_dash_ratio 12.000000)
 			(dashed_line_gap_ratio 3.000000)
@@
 			(plotinvisibletext no)
 			(sketchpadsonfab no)
-			(subtractmaskfromsilk no)
+			(subtractmaskfromsilk yes)
 			(outputformat 1)
 			(mirror no)
-			(drillshape 1)
+			(drillshape 0)
 			(scaleselection 1)
-			(outputdirectory "")
+			(outputdirectory "gerbers/")
 		)
 	)
@@
 		)
 	)
-	(footprint "adhoc:MountingHole_1.8mm_M1.6"
+	(footprint "adhoc:MountingHole_1.7mm_M1.6"
 		(layer "F.Cu")
 		(at 121.5 79.5)
@@
 			)
 		)
-		(property "Footprint" "adhoc:MountingHole_1.8mm_M1.6"
+		(property "Footprint" "adhoc:MountingHole_1.7mm_M1.6"
 			(at 0 0 0)
 			(unlocked yes)
@@
 		(pad "" np_thru_hole circle
 			(at 0 0)
-			(size 1.8 1.8)
-			(drill 1.8)
-			(layers "F&B.Cu" "*.Mask")
+			(size 1.7 1.7)
+			(drill 1.7)
+			(layers "F&B.Cu" "*.Paste" "*.Mask")
 		)
 	)
@@
 		)
 	)
-	(footprint "adhoc:MountingHole_1.8mm_M1.6"
+	(footprint "adhoc:MountingHole_1.7mm_M1.6"
 		(layer "F.Cu")
 		(at 121.5 52.5)
@@
 			)
 		)
-		(property "Footprint" "adhoc:MountingHole_1.8mm_M1.6"
+		(property "Footprint" "adhoc:MountingHole_1.7mm_M1.6"
 			(at 0 0 0)
 			(unlocked yes)
@@
 		(pad "" np_thru_hole circle
 			(at 0 0)
-			(size 1.8 1.8)
-			(drill 1.8)
-			(layers "F&B.Cu" "*.Mask")
+			(size 1.7 1.7)
+			(drill 1.7)
+			(layers "F&B.Cu" "*.Paste" "*.Mask")
 		)
 	)
@@
 		)
 	)
-	(footprint "adhoc:MountingHole_1.8mm_M1.6"
+	(footprint "adhoc:MountingHole_1.7mm_M1.6"
 		(layer "F.Cu")
 		(at 102.5 79.5)
@@
 			)
 		)
-		(property "Footprint" "adhoc:MountingHole_1.8mm_M1.6"
+		(property "Footprint" "adhoc:MountingHole_1.7mm_M1.6"
 			(at 0 0 0)
 			(unlocked yes)
@@
 		(pad "" np_thru_hole circle
 			(at 0 0)
-			(size 1.8 1.8)
-			(drill 1.8)
-			(layers "F&B.Cu" "*.Mask")
+			(size 1.7 1.7)
+			(drill 1.7)
+			(layers "F&B.Cu" "*.Paste" "*.Mask")
 		)
 	)
