File: Tiramisu.kicad_sch (KiCad schematic)
At the start: 26 parts, among them J1 Conn_ARM_SWD_TagConnect_TC203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, J2 USB_C_Receptacle_USB2.0_16P, Q1 Q_PMOS_GSD, U1 MDBT50Q-1MV2, U2 LSM6DSV, U3 MCP73831-2-OT

Commit message: that should be a +3V3 route oops
Connections:
- net +3.3V: now also J1.1 (VCC)
- net VCC: no longer J1.1 (VCC)
Changed lines of the file:
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@@
+	)
+	(symbol
+		(lib_name "+3.3V_1")
+		(lib_id "power:+3.3V")
+		(at 62.23 22.86 0)
+		(unit 1)
+		(exclude_from_sim no)
+		(in_bom yes)
+		(on_board yes)
+		(dnp no)
+		(fields_autoplaced yes)
+		(property "Reference" "#PWR06"
+			(at 62.23 26.67 0)
+			(effects
+				(font
+					(size 1.27 1.27)
+				)
+				(hide yes)
+			)
+		)
+		(property "Value" "+3.3V"
+			(at 62.23 17.78 0)
+			(effects
+				(font
+					(size 1.27 1.27)
+				)
+			)
+		)
+		(property "Footprint" ""
+			(at 62.23 22.86 0)
+			(effects
+				(font
+					(size 1.27 1.27)
+				)
+				(hide yes)
+			)
+		)
+		(property "Datasheet" ""
+			(at 62.23 22.86 0)
+			(effects
+				(font
+					(size 1.27 1.27)
+				)
+				(hide yes)
+			)
+		)
+		(property "Description" "Power symbol creates a global label with name \"+3.3V\""
+			(at 62.23 22.86 0)
+			(effects
+				(font
+					(size 1.27 1.27)
+				)
+				(hide yes)
+			)
+		)
+		(pin "1"
+		)
+		(instances
+			(project "Tiramisu"
+				(path "/0001b6d0-4607-4d14-8fe0-154bb94236d5"
+					(reference "#PWR06")
+					(unit 1)
+				)
+			)
+		)
 	)
 	(symbol
@@
 					(unit 1)
 				)
-			)
-		)
-	)
-	(symbol
-		(lib_id "power:VCC")
-		(at 62.23 22.86 0)
-		(unit 1)
-		(exclude_from_sim no)
-		(in_bom yes)
-		(on_board yes)
-		(dnp no)
-		(fields_autoplaced yes)
-		(property "Reference" "#PWR06"
-			(at 62.23 26.67 0)
-			(effects
-				(font
-					(size 1.27 1.27)
-				)
-				(hide yes)
-			)
-		)
-		(property "Value" "VCC"
-			(at 62.23 17.78 0)
-			(effects
-				(font
-					(size 1.27 1.27)
-				)
-			)
-		)
-		(property "Footprint" ""
-			(at 62.23 22.86 0)
-			(effects
-				(font
-					(size 1.27 1.27)
-				)
-				(hide yes)
-			)
-		)
-		(property "Datasheet" ""
-			(at 62.23 22.86 0)
-			(effects
-				(font
-					(size 1.27 1.27)
-				)
-				(hide yes)
-			)
-		)
-		(property "Description" "Power symbol creates a global label with name \"VCC\""
-			(at 62.23 22.86 0)
-			(effects
-				(font
-					(size 1.27 1.27)
-				)
-				(hide yes)
-			)
-		)
-		(pin "1"
-		)
-		(instances
-			(project "Tiramisu"
-				(path "/0001b6d0-4607-4d14-8fe0-154bb94236d5"
-					(reference "#PWR06")
-					(unit 1)
-				)

Commit message: final export
Parts:
- H1, H2, H3: footprint adhoc:MountingHole_1.8mm_M1.6 -> adhoc:MountingHole_1.7mm_M1.6
Changed lines of the file:
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@@
 			)
 		)
-		(property "Footprint" "adhoc:MountingHole_1.8mm_M1.6"
+		(property "Footprint" "adhoc:MountingHole_1.7mm_M1.6"
 			(at 157.48 151.13 0)
 			(effects
@@
 			)
 		)
-		(property "Footprint" "adhoc:MountingHole_1.8mm_M1.6"
+		(property "Footprint" "adhoc:MountingHole_1.7mm_M1.6"
 			(at 157.48 146.05 0)
 			(effects
@@
 			)
 		)
-		(property "Footprint" "adhoc:MountingHole_1.8mm_M1.6"
+		(property "Footprint" "adhoc:MountingHole_1.7mm_M1.6"
 			(at 157.48 156.21 0)
 			(effects
